Commit message: Source for lesson 3,4

File: urdf/rosbots.xacro (robot description, xacro)
@@ -381,4 +381,23 @@
         </geometry>
         <origin rpy="0.0 0 0" xyz="0 0 0.0"/>
+      </collision>
+    </link>
+    <joint name="camera_joint" type="fixed">
+      <origin xyz="0.49 -0.03 0.75" rpy="0 0.21 0" />
+      <parent link="base_link"/>
+      <child link="camera_link" />
+    </joint>
+    <link name="camera_link">
+      <visual>
+        <geometry>
+          <mesh filename="package://MAC-design-and-operation/meshes/camera.dae" scale="4.0 4.0 4.0"/>
+        </geometry>
+        <origin xyz="0.0 0 0" rpy="0 0 0"/>
+      </visual>
+      <collision>
+        <geometry>
+          <mesh filename="package://MAC-design-and-operation/meshes/camera.dae" scale="4.0 4.0 4.0"/>
+        </geometry>
+        <origin xyz="0.0 0 0" rpy="0 0 0"/>
       </collision>
     </link>
@@ -403,3 +422,34 @@
     </plugin>
   </gazebo>
+  <gazebo reference="camera_link">
+    <sensor type="camera" name="camera1">
+      <update_rate>30.0</update_rate>
+      <camera name="head">
+        <horizontal_fov>1.04</horizontal_fov>
+        <image>
+          <width>320</width>
+          <height>240</height>
+          <format>R8G8B8</format>
+        </image>
+        <clip>
+          <near>0.1</near>
+          <far>50</far>
+        </clip>
+      </camera>
+      <plugin name="camera_controller" filename="libgazebo_ros_camera.so">
+        <alwaysOn>true</alwaysOn>
+        <updateRate>0</updateRate>
+        <cameraName>camera1</cameraName>
+        <imageTopicName>image_raw</imageTopicName>
+        <cameraInfoTopicName>camera_info</cameraInfoTopicName>
+        <frameName>camera</frameName>
+        <hackBaseline>0.07</hackBaseline>
+        <distortionK1>0.0</distortionK1>
+        <distortionK2>0.0</distortionK2>
+        <distortionK3>0.0</distortionK3>
+        <distortionT1>0.0</distortionT1>
+        <distortionT2>0.0</distortionT2>
+      </plugin>
+    </sensor>
+  </gazebo>
 </robot>

Commit message: Lessons 5,6

File: urdf/rosbots.xacro (robot description, xacro)
@@ -453,3 +453,59 @@
     </sensor>
   </gazebo>
+  <joint name="hokuyo_joint" type="fixed">
+	  <origin xyz="0.49 -0.1 0.75" rpy="0 0.21 0" />
+	  <parent link="base_link"/>
+	  <child link="hokuyo_link"/>
+	</joint>
+	<link name="hokuyo_link">
+	  <visual>
+	      <origin xyz="0 0 0" rpy="0 0 0"/>
+	      <geometry>
+		<mesh filename="package://MAC-design-and-operation/meshes/hokuyo.dae"/>
+	      </geometry>
+	    </visual>
+	  <collision>
+	    <geometry>
+	      <mesh filename="package://MAC-design-and-operation/meshes/hokuyo.dae"/>
+	      <box size="0.1 0.1 0.1"/>
+	    </geometry>
+	    <origin xyz="0.0 0 0" rpy="0 0 0"/>
+	  </collision>
+	</link>
+	<!-- hokuyo -->
+	  <gazebo reference="hokuyo_link">
+	    <sensor type="gpu_ray" name="head_hokuyo_sensor">
+	      <pose>0 0 0 0 0 0</pose>
+	      <visualize>false</visualize>
+	      <update_rate>40</update_rate>
+	      <ray>
+		<scan>
+		  <horizontal>
+		    <samples>720</samples>
+		    <resolution>1</resolution>
+		    <min_angle>-1.570796</min_angle>
+		    <max_angle>1.570796</max_angle>
+		  </horizontal>
+		</scan>
+		<range>
+		  <min>0.10</min>
+		  <max>30.0</max>
+		  <resolution>0.01</resolution>
+		</range>
+		<noise>
+		  <type>gaussian</type>
+		  <!-- Noise parameters based on published spec for Hokuyo laser
+		       achieving "+-30mm" accuracy at range < 10m.  A mean of 0.0m and
+		       stddev of 0.01m will put 99.7% of samples within 0.03m of the true
+		       reading. -->
+		  <mean>0.0</mean>
+		  <stddev>0.01</stddev>
+		</noise>
+	      </ray>
+	      <plugin name="gazebo_ros_head_hokuyo_controller" filename="libgazebo_ros_gpu_laser.so">
+		<topicName>/bot_0/laser/scan</topicName>
+		<frameName>hokuyo_link</frameName>
+	      </plugin>
+	    </sensor>
+	  </gazebo>
 </robot>
