Commit message: Added models for last practice

File: urdf/rosbots_0.xacro (robot description, xacro)
@@ -384,5 +384,5 @@
   </link>
 	<joint name="hokuyo_joint" type="fixed">
-	  <origin xyz="0.49 -0.1 0.75" rpy="0 0.21 0" />
+	  <origin xyz="0.49 -0.1 0.75" rpy="0 0 0" />
 	  <parent link="base_link"/>
 	  <child link="hokuyo_link"/>

File: urdf/rosbots_1.xacro (robot description, xacro)
@@ -384,5 +384,5 @@
   </link>
 	<joint name="hokuyo_joint" type="fixed">
-	  <origin xyz="0.49 -0.1 0.75" rpy="0 0.21 0" />
+	  <origin xyz="0.49 -0.1 0.75" rpy="0 0 0" />
 	  <parent link="base_link"/>
 	  <child link="hokuyo_link"/>

File: urdf/rosbots_2.xacro (robot description, xacro)
@@ -384,5 +384,5 @@
   </link>
 	<joint name="hokuyo_joint" type="fixed">
-	  <origin xyz="0.49 -0.1 0.75" rpy="0 0.21 0" />
+	  <origin xyz="0.49 -0.1 0.75" rpy="0 0 0" />
 	  <parent link="base_link"/>
 	  <child link="hokuyo_link"/>
